File: hardware/cdi-board/TopVVtester.sch (KiCad schematic (older format))
At the start: 79 parts, among them P1 VR IN, P3 COIL, P35 HOLE, P4 12v in, P5 GEN A, P52 VR1_out select, P64 HOLE, P65 HOLE, P66 HOLE, P67 HOLE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

Commit message: cdi-board: MAC-10.0 Test Board
Imported from original project folder:
  FPGA_TopVtester

31 files changed, 48282 insertions(+), 29014 deletions(-)
Parts:
- removed C1, C3: 100nF, symbol C
- removed C11: 0.022uF, symbol CP_US
- removed C13: CP_US, symbol CP_US
- removed C4, C5: 0.47uF 275VAC, symbol C
- removed D1, D2, D4: 1N5408, symbol DIODE
- removed D3: 1N4004, symbol DIODE
- removed D5: RURG3060, symbol RURG3060
- removed L1: PCV-2-394-05L, ~, symbol INDUCTOR
- removed P35, P64, P65, P66, P67, P68: HOLE, symbol CONN_1
- removed Q1: FCA47N60, TO-3PN, symbol FCA47N60
- removed R18: 15K 0.25W, symbol R
- removed R19: 1M 0.25W 2%, symbol R
- removed R20: 10K 0.25W 2%, symbol R
- removed R6: 1M 0.25W, symbol R
- removed R8: 100 0.5W, symbol R
- removed SCR1: BT151, symbol THYRISTOR
- removed TH1: NTC, symbol THERMISTOR
- removed U3: LM393, symbol LM393
- removed U8: POWER_SELECT, ~, symbol POWER_SELECT
- removed U9: KILL SEL, ~, symbol POWER_SELECT2
- added C1: 0.01uF, symbol CP_US
- added P2: VR IN, ~, symbol CONN_2
- added P6: CAS1, ~, symbol CONN_2
- added P7: FPGA 48, ~, symbol CONN_2
- added T1: -NPN-TO92, transistor-TO92, symbol -NPN-TO92
- added VR3: 50K Variable, symbol VR1
- C2: value 10uF 25V -> 0.01uF; footprint (none) -> ~
- C7: value 0.01uF -> 0.33uF
- P3: value COIL -> cdi trig
- P4: value 12v in -> opto out
- P5: value GEN A -> 555 out
- R17: value 10K 0.25W -> 1K3 0.25W
- R3: value 51ohm 0.25W -> 1K 0.25W
- R5: value 1M 0.25W -> 100 ohm 0.25W
- VR1: value 10K Variable -> 1M Variable
Connections:
- net 150VGenA is gone; now on net 555output: P5.1 (P1)
- net +8Vi: no longer P4.1 (P1)
- net CAS1: now also U10.15 (B3), P6.1 (P1)
- net CDI_Trigger: now also P3.1 (P1), U10.9 (A7); no longer U10.11 (B7)
- net FPGA_48: now also U10.5 (A3), P7.1 (P1)
- net FPGA_59: now also U10.2 (A0); no longer U10.18 (B0)
- net FPGA_61: now also U10.17 (B1); no longer U10.3 (A1)
- net FPGA_62: now also U10.16 (B2); no longer U10.4 (A2)
- net FPGA_65: now also U10.11 (B7); no longer U10.9 (A7)
- net GND: now also C2.2, P4.2 (PM), C1.2, P6.2 (PM), P7.2 (PM), T1.1 (E); no longer VR1.1
- net KtypeCS_0: now also U10.4 (A2); no longer U10.16 (B2)
- net KtypeSCK: now also U10.3 (A1); no longer U10.17 (B1)
- net KtypeSO: now also U10.18 (B0); no longer U10.2 (A0)
- net V5.0: now also C2.1, R5.2, U7.4 (R), VR3.1; no longer VR1.3
- net at P1.1 (P1), R71.2: now also P2.2 (PM)
- net 555output: now reaches R5.1
- net 555output: now also P2.1 (P1), T1.3 (C)
- net at R2.2, U1.4 (E): now also P4.1 (P1); no longer R3.1
- net at R4.2: now also VR1.2, VR1.3; no longer C2.1
- net at R17.1, U7.2 (TR), U7.6 (THR): now also C7.1
- net at R17.2, U7.7 (DIS): now also R4.1
- net at U7.3 (OUT): now also R3.1
- net at U7.5 (CV): now also C1.1; no longer C7.1
- new net: VR1.1, VR3.2, VR3.3
- new net: R3.2, T1.2 (B)
Other:
- note added: "ERROR:\nAdd 1K resistor here"
- note added: "ERROR:\nMake 100K VR here"
- note added: "Optional:\nLeave open if no\ncurrent limit needed"
- note removed: "+ ignition coil"
- note removed: "Generator Coil"
- note removed: "Kill Switch"
- note removed: "Optional"
- note removed: "PCB MOUNTING HOLES"
- moved on the sheet: C10, C6, C7, C8, R17, U7, VR1
