File: hardware/cdi-board/TopVVtester3.sch (KiCad schematic (older format))
At the start: 91 parts, among them P1 CONN_1, P2 CONN_10X2, P2.1 CONN_10X2, P20 CONN_1, P21 CONN_1, P22 CONN_1, P23 CONN_1, P24 CONN_1, P28 CONN_1, P29 CONN_1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

Commit message: cdi-board: TopB 3 (silkscreen REV 3.0)
Imported from original project folder:
  FPGA_TopVtester3

22 files changed, 34061 insertions(+), 134143 deletions(-)
Parts:
- removed P2, P2.1: CONN_10X2, symbol CONN_10X2
- removed P6, P9: CONN_1, symbol CONN_1
- added C12: 10 uF, symbol CP
- added P26, P27: CONN_1, symbol CONN_1
- renumbered P5 to P2
Connections:
- net +8Vi: now also C12.1
- net GND: now also C12.2
- net VRIN1+: now also P26.1
- net VRIN1-: now also P27.1
Other:
- note added: "NOTE: 15-01-2017 this \ndiode "D1" is around\n the wrong way"
- moved on the sheet: U2, U4
