File: hardware/cdi-board/TopVVtester2.sch (KiCad schematic (older format))
At the start: 90 parts, among them P1 CONN_1, P2 CONN_1, P20 CONN_1, P21 CONN_1, P22 CONN_1, P23 CONN_1, P24 CONN_1, P26 CONN_1, P27 CONN_1, P28 CONN_1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

Commit message: cdi-board: TopB 2 (silkscreen REV 1.0) - BOM
Imported from original project folder:
  FPGA_TopVtester2

29 files changed, 613294 insertions(+), 23130 deletions(-)
Other:
- note added: "NOTE: 15-01-2017 \nD1 and D2 increase foot print\nhole diamater"
- note added: "NOTE: 15-01-2017 \nD3 foot print incorrect"
- note added: "NOTE: 15-01-2017 \nopto isolator circuit does not work,\nthis needs to be revisited on the next revision.\n\nusing T2 and R24 works to give signal to R3"
- note added: "NOTE: 15-01-2017 this\nC2 should be polar cap\nwith -ve toward SCR"
- note added: "NOTE: 15-01-2017 this\nC3 should be 10nF &\nnon polar footprint"
- note added: "NOTE: 15-01-2017 this\nDiode "D1" is around\nthe wrong way."
- note removed: "NOTE: 15-01-2017 this \ndiode "D1" is around\n the wrong way"
Changed lines of the file:
@@
 LIBS:wildcard88
 LIBS:ANTS_MOD1
-LIBS:TopVVtester3-cache
+LIBS:TopVVtester2-cache
 EELAYER 27 0
 EELAYER END
@@
 Sheet 1 1
 Title ""
-Date "15 jan 2017"
+Date "16 jan 2017"
 Rev ""
 Comp ""
@@
 	1    0    0    -1
 $EndComp
-Text Notes 14400 8150 0    60   ~ 0
-NOTE: 15-01-2017 this \ndiode "D1" is around\n the wrong way
+Text Notes 14750 8150 0    60   ~ 0
+NOTE: 15-01-2017 this\nDiode "D1" is around\nthe wrong way.
+Text Notes 13950 10500 0    60   ~ 0
+NOTE: 15-01-2017 \nopto isolator circuit does not work,\nthis needs to be revisited on the next revision.\n\nusing T2 and R24 works to give signal to R3
+Text Notes 18350 9150 0    60   ~ 0
+NOTE: 15-01-2017 this\nC3 should be 10nF &\nnon polar footprint
+Text Notes 16650 9200 0    60   ~ 0
+NOTE: 15-01-2017 \nD3 foot print incorrect
+Text Notes 15850 7150 0    60   ~ 0
+NOTE: 15-01-2017 \nD1 and D2 increase foot print\nhole diamater
+Text Notes 17600 7200 0    60   ~ 0
+NOTE: 15-01-2017 this\nC2 should be polar cap\nwith -ve toward SCR
+Wire Notes Line
+	18000 7450 18000 7800
+Wire Notes Line
+	18000 7800 17650 7800
+Wire Notes Line
+	18550 8550 18700 8550
+Wire Notes Line
+	18700 8550 18700 9050
+Wire Notes Line
+	16900 8700 16900 9100
+Wire Notes Line
+	16900 9100 16850 9100
+Wire Notes Line
+	15450 7950 15200 7950
+Wire Notes Line
+	15200 7950 15200 8050
+Wire Notes Line
+	16600 7250 16600 7950
+Wire Notes Line
+	16600 7500 16050 7500
+Wire Notes Line
+	16600 7950 15750 7950
+Wire Notes Line
+	13900 9050 16050 9050
+Wire Notes Line
+	16050 9050 16050 10300
+Wire Notes Line
+	16050 10300 13900 10300
+Wire Notes Line
+	13900 10300 13900 9050
+Wire Notes Line
+	15100 10300 15100 10450
 $EndSCHEMATC

Commit message: cdi-board: TopB 2 - reduced CDI experiment
Imported from original project folder:
  FPGA_TopVtester2 - Copy

2 files changed, 72 insertions(+), 768 deletions(-)
Parts:
- removed C19: 0.1uF, symbol C
- removed C2: 10uF 25V, symbol C
- removed D1: 1N5408, symbol DIODE
- removed D6, D7, D8, D9: 1N4004, symbol DIODE
- removed P1, P2, P22, P23, P24: CONN_1, symbol CONN_1
- removed P7: CONN_3, ~, symbol CONN_3
- removed R1, R24: 330 0.25W, symbol R
- removed R2: 4K7 0.25W, symbol R
- removed R20: 10K, symbol R
- removed T2: ^^NPN-SOT23, ~, symbol ^^NPN-SOT23
- removed U1: 4N25, symbol OPTO-TRANSISTOR
- removed U10: 74LVC245, ~, symbol 74LVC245
- removed U7: MAX6816, symbol MAX6816
- removed U8: HV SEL, ~, symbol POWER_SELECT
- added Rx: res, symbol R
- C3: value 100nF -> 10nF
Connections:
- net labels added: +12V
- net labels removed: 150VGenA, 150VGenB, CDI_Trigger, FPGA_48, FPGA_50, FPGA_51, FPGA_55, GENA, GENB, HV_00
- wire segments 324 -> 250
Other:
- note added: "+150 to 250V DC"
- note added: "CDI Trigger\n"
- note added: "COIL"
- note added: "Could be removed"
- note added: "OPTION 1"
- note added: "OPTION 2"
- note removed: "<------"
- note removed: "NOTE: 15-01-2017 \nD1 and D2 increase foot print\nhole diamater"
- note removed: "NOTE: 15-01-2017 \nD3 foot print incorrect"
- note removed: "NOTE: 15-01-2017 \nopto isolator circuit does not work,\nthis needs to be revisited on the next revision.\n\nusing T2 and R24 works to give signal to R3"
- note removed: "NOTE: 15-01-2017 this\nC2 should be polar cap\nwith -ve toward SCR"
- note removed: "NOTE: 15-01-2017 this\nC3 should be 10nF &\nnon polar footprint"
- note removed: "NOTE: 15-01-2017 this\nDiode "D1" is around\nthe wrong way."
- note removed: "from HV Generator Coil"
