File: hardware/logic-board/S6LX9_R2.sch (KiCad schematic (older format))
At the start: 112 parts, among them P15 DC IN, P2 CONN_10X2, P20 XILINX CABLE, P5 PIC_ISP, P6 CONN_1, P7 CONN_1, P8 CONN_10X2, Q1 ^^NPN-SOT23, Q2 ^^NPN-SOT23, Q5 ^^NPN-BC817-SOT323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

Commit message: logic-board: S6LX9 R2 layout routing
Imported from original project folder:
  backup 12-10-2015 2333

6 files changed, 2479 insertions(+), 2082 deletions(-)
Parts:
- added P1: CONN_4X2, ~, symbol CONN_4X2
Connections:
- wire segments 929 -> 936
Changed lines of the file:
@@
 Text Label 22900 13750 2    60   ~ 0
 FPGA_114
-Text Label 22250 11100 2    60   ~ 0
+Text Label 26900 7800 2    60   ~ 0
 FPGA_112
-Text Label 8450 7900 0    60   ~ 0
+Text Label 26900 7700 2    60   ~ 0
 FPGA_111
 Text Label 14450 13850 0    60   ~ 0
@@
 Text Label 14450 13250 0    60   ~ 0
 FPGA_118
-Text Label 12200 7750 2    60   ~ 0
+Text Label 11850 6950 0    60   ~ 0
 FPGA_132
 Text Label 9500 26850 2    60   ~ 0
@@
 Text Label 14450 12350 0    60   ~ 0
 FPGA_132
-Text Label 12200 6150 2    60   ~ 0
+Text Label 11850 7050 0    60   ~ 0
 FPGA_133
 Text Label 40350 15000 2    60   ~ 0
@@
 	22250 11400 22600 11400
 Wire Wire Line
-	22250 11100 22600 11100
-Wire Wire Line
 	4650 11850 7900 11850
 Wire Wire Line
@@
 	22250 12300 22600 12300
 Wire Wire Line
-	22150 10800 22600 10800
-Wire Wire Line
 	23700 12300 23600 12300
 Connection ~ 23700 12000
@@
 	40050 19650 40600 19650
 Wire Wire Line
-	41800 18050 42200 18050
+	40450 18050 42200 18050
 Wire Wire Line
-	40050 19150 40150 19150
-Wire Wire Line
-	40150 19150 40150 20750
+	40050 19150 40450 19150
 Wire Wire Line
 	40050 19550 40150 19550
-Connection ~ 40150 19550
 Wire Wire Line
 	38650 19550 38450 19550
@@
 	29850 19350 30100 19350
 Wire Wire Line
-	40150 20750 40750 20750
-Wire Wire Line
 	44350 23000 44150 23000
 Wire Wire Line
@@
 	44550 18400 44900 18400
 Connection ~ 41950 18150
-Wire Wire Line
-	41800 21750 41800 18050
 $Comp
 L R R39
@@
 Text Notes 34500 20700 0    60   ~ 0
 FOR RUN/FLASH
-Text Label 40750 20750 0    60   ~ 0
-FLASH_CS
 Wire Wire Line
 	40350 21750 41800 21750
@@
 Text Notes 14900 13750 0    60   ~ 0
 to LED4
-Text Notes 21800 11100 2    60   ~ 0
-to LED4
 Text Notes 21800 11400 2    60   ~ 0
 to LED3
@@
 Text Label 13500 8400 2    60   ~ 0
 FPGA_67
-Text Notes 21600 10800 2    60   ~ 0
-to LED5
 Text Notes 15050 15550 2    60   ~ 0
 to LED5
@@
 Text Notes 37000 14300 0    60   ~ 0
 FPGA Pin 121 socz80 UART CTS - input to fpga\nFPGA Pin 119 socz80 UART RTS - output from fpga\nFPGA Pin 120 socz80 UART RX - input to fpga\nFPGA Pin 118 socz80 UART TX - output from fpga
-Text Label 22150 10800 2    60   ~ 0
+Text Label 13250 7100 2    60   ~ 0
 FPGA_100
 Text Label 2550 12500 0    60   ~ 0
@@
 Wire Wire Line
 	40750 15200 40750 15000
+Wire Wire Line
+	40450 19150 40450 18050
+Connection ~ 40150 19150
+Wire Wire Line
+	40150 19550 40150 19150
+Text Label 26900 7900 2    60   ~ 0
+FPGA_114
+Text Label 26900 8000 2    60   ~ 0
+FPGA_115
+Text Label 27900 7700 0    60   ~ 0
+FPGA_116
+Text Label 27900 7800 0    60   ~ 0
+FPGA_117
+Wire Wire Line
+	27000 7700 26900 7700
+Wire Wire Line
+	26900 7800 27000 7800
+Wire Wire Line
+	27000 7900 26900 7900
+Wire Wire Line
+	26900 8000 27000 8000
+Wire Wire Line
+	27800 7700 27900 7700
+Wire Wire Line
+	27900 7800 27800 7800
+Wire Wire Line
+	11750 6950 11850 6950
+Wire Wire Line
+	11850 7050 11750 7050
+$Comp
+L CONN_4X2 P1
+U 1 1 561BD723
+P 27400 7850
+F 0 "P1" H 27400 8100 50  0000 C CNN
+F 1 "CONN_4X2" V 27400 7850 40  0000 C CNN
+F 2 "~" H 27400 7850 60  0000 C CNN
+F 3 "~" H 27400 7850 60  0000 C CNN
+	1    27400 7850
+	1    0    0    -1
+$EndComp
+Text Label 28000 8000 0    60   ~ 0
++8Vi
+Text Label 28000 7900 0    60   ~ 0
+GND
+Wire Wire Line
+	28000 7900 27800 7900
+Wire Wire Line
+	27800 8000 28000 8000
 $EndSCHEMATC

Commit message: logic-board: S6LX9 R2 schematic and layout updates
Imported from original project folder:
  19-02-2016 1257

6 files changed, 7256 insertions(+), 2460 deletions(-)
Parts:
- removed P1: CONN_4X2, ~, symbol CONN_4X2
- removed SW1: RESET, symbol SW_PUSH
- added P1: FPGA PINS, symbol CONN_4
- added R14: 1K, symbol R
- added U7: M25P80, symbol M25P80
Connections:
- wire segments 936 -> 950
Other:
- note added: "25Pxx Serial Flash 2"
- note added: "to Flash 2"
- note removed: "console select ->\npull to GND to make\nthis system console"
- note removed: "to LED4"
Changed lines of the file:
@@
 Sheet 1 1
 Title "noname.sch"
-Date "12 oct 2015"
+Date "8 feb 2016"
 Rev ""
 Comp ""
@@
 	-1   0    0    -1
 $EndComp
-Text Label 11600 8500 0    60   ~ 0
-FPGA_48
 Text Label 12050 30300 2    60   ~ 0
 FPGA_46
@@
 Text Label 28750 18600 2    60   ~ 0
 FPGA_58
-Text Label 11600 8200 0    60   ~ 0
-FPGA_57
-Text Label 11600 8300 0    60   ~ 0
-FPGA_56
-Text Label 11600 8400 0    60   ~ 0
-FPGA_55
 NoConn ~ 5850 23600
 NoConn ~ 5850 21700
@@
 Text Label 22900 13750 2    60   ~ 0
 FPGA_114
-Text Label 26900 7800 2    60   ~ 0
+Text Label 26050 8300 2    60   ~ 0
 FPGA_112
-Text Label 26900 7700 2    60   ~ 0
-FPGA_111
 Text Label 14450 13850 0    60   ~ 0
 FPGA_111
@@
 Text Label 14450 13250 0    60   ~ 0
 FPGA_118
-Text Label 11850 6950 0    60   ~ 0
-FPGA_132
 Text Label 9500 26850 2    60   ~ 0
 FPGA_131
@@
 Text Label 14450 12350 0    60   ~ 0
 FPGA_132
-Text Label 11850 7050 0    60   ~ 0
-FPGA_133
-Text Label 40350 15000 2    60   ~ 0
+Text Label 14300 8450 2    60   ~ 0
 FPGA_134
 Text Label 12050 30200 2    60   ~ 0
@@
 Text Label 13700 29100 0    60   ~ 0
 FPGA_9
-Text Label 10300 7100 2    60   ~ 0
-FPGA_8
-Text Label 10300 7200 2    60   ~ 0
-FPGA_7
 Text Label 13700 30800 0    60   ~ 0
 FPGA_6
@@
 Text Label 6150 22200 0    60   ~ 0
 FPGA_66
-Text Label 14900 6900 0    60   ~ 0
+Text Label 26050 8000 2    60   ~ 0
 FPGA_67
-Text Label 14900 7000 0    60   ~ 0
-FPGA_66
 Wire Wire Line
 	6150 22100 5850 22100
@@
 Wire Wire Line
 	14050 17450 14250 17450
-Text Label 14900 7100 0    60   ~ 0
+Text Label 26050 8200 2    60   ~ 0
 FPGA_75
-Text Label 13850 6450 0    60   ~ 0
+Text Label 26050 8100 2    60   ~ 0
 FPGA_74
 Text Label 2750 -5100 0    60   ~ 0
@@
 Text Notes 32900 20600 0    60   ~ 0
 Q2 out is LOW on PowerUp
-$Comp
-L SW_PUSH SW1
-U 1 1 54A764C1
-P 29650 18600
-F 0 "SW1" H 29800 18710 50  0000 C CNN
-F 1 "RESET" H 29650 18520 50  0000 C CNN
-F 2 "" H 29650 18600 60  0001 C CNN
-F 3 "" H 29650 18600 60  0001 C CNN
-	1    29650 18600
-	0    -1   -1   0
-$EndComp
 Text Label 29750 18250 0    60   ~ 0
 GND
@@
 Wire Wire Line
 	6150 22600 5850 22600
-Text Label 8450 6950 0    60   ~ 0
-FPGA_61
-Text Label 8450 6850 0    60   ~ 0
-FPGA_62
 Text Label 9400 23650 2    60   ~ 0
 FPGA_64
@@
 Wire Wire Line
 	43500 7400 44450 7400
-Text Label 10350 8550 0    60   ~ 0
-FPGA_50
-Text Label 10350 8450 0    60   ~ 0
-FPGA_51
 Text Label 40950 14500 0    60   ~ 0
 TX_SOUT
@@
 Text Notes 41400 14300 0    60   ~ 0
 Pin 3 (RTS) - OUTPUT from FT232\nPin 11 (CTS) - INPUT to FT232\n
-Text Notes 39050 15000 0    60   ~ 0
-console select ->\npull to GND to make\nthis system console
-Wire Wire Line
-	40350 15000 40750 15000
-Text Label 40450 15200 2    60   ~ 0
-GND
-Wire Wire Line
-	40450 15200 40750 15200
 Wire Wire Line
 	39950 14300 40950 14300
@@
 SOFT RESET
 Text Notes 14900 13750 0    60   ~ 0
-to LED4
+to Flash 2
 Text Notes 21800 11400 2    60   ~ 0
 to LED3
@@
 Text Label 39550 24250 2    60   ~ 0
 FPGA_132
-Text Label 13500 8400 2    60   ~ 0
-FPGA_67
 Text Notes 15050 15550 2    60   ~ 0
 to LED5
@@
 Text Notes 37000 14300 0    60   ~ 0
 FPGA Pin 121 socz80 UART CTS - input to fpga\nFPGA Pin 119 socz80 UART RTS - output from fpga\nFPGA Pin 120 socz80 UART RX - input to fpga\nFPGA Pin 118 socz80 UART TX - output from fpga
-Text Label 13250 7100 2    60   ~ 0
-FPGA_100
-Text Label 2550 12500 0    60   ~ 0
+Text Label 4350 12300 0    60   ~ 0
 VCCINT
-Text Label 2500 12050 0    60   ~ 0
+Text Label 4500 11600 0    60   ~ 0
 VCCAUX
-Text Label 2550 13300 0    60   ~ 0
+Text Label 4400 12900 0    60   ~ 0
 VCC0_0
-Text Label 2500 13600 0    60   ~ 0
+Text Label 4350 13450 0    60   ~ 0
 VCC0_1
-Text Label 2500 14050 0    60   ~ 0
+Text Label 4400 13850 0    60   ~ 0
 VCC0_2
-Text Label 2500 14350 0    60   ~ 0
+Text Label 4400 14200 0    60   ~ 0
 VCC0_3
 Wire Wire Line
@@
 OLD: flash select button
 Wire Wire Line
-	40750 15200 40750 15000
-Wire Wire Line
 	40450 19150 40450 18050
 Connection ~ 40150 19150
 Wire Wire Line
 	40150 19550 40150 19150
-Text Label 26900 7900 2    60   ~ 0
+Text Label 30700 27500 2    60   ~ 0
 FPGA_114
-Text Label 26900 8000 2    60   ~ 0
+Text Label 30700 27600 2    60   ~ 0
 FPGA_115
-Text Label 27900 7700 0    60   ~ 0
+Text Label 33650 28000 0    60   ~ 0
 FPGA_116
-Text Label 27900 7800 0    60   ~ 0
+Text Label 33650 28100 0    60   ~ 0
 FPGA_117
 Wire Wire Line
-	27000 7700 26900 7700
+	26050 8300 26300 8300
 Wire Wire Line
-	26900 7800 27000 7800
+	30700 27500 31300 27500
 Wire Wire Line
-	27000 7900 26900 7900
+	30700 27600 31300 27600
 Wire Wire Line
-	26900 8000 27000 8000
+	33100 28000 33650 28000
 Wire Wire Line
-	27800 7700 27900 7700
+	33050 28100 33650 28100
+$Comp
+L M25P80 U7
+U 1 1 56A1E9B3
+P 31900 27650
+F 0 "U7" H 31900 27650 60  0000 C CNN
+F 1 "M25P80" H 32000 27550 60  0000 C CNN
+F 2 "" H 31900 27650 60  0000 C CNN
+F 3 "" H 31900 27650 60  0000 C CNN
+	1    31900 27650
+	1    0    0    -1
+$EndComp
+Text Label 33950 27250 0    60   ~ 0
+V3.3
+$Comp
+L R R14
+U 1 1 56A1E9D0
+P 33350 27600
+F 0 "R14" V 33430 27600 50  0000 C CNN
+F 1 "1K" V 33350 27600 50  0000 C CNN
+F 2 "" H 33350 27600 60  0001 C CNN
+F 3 "" H 33350 27600 60  0001 C CNN
+	1    33350 27600
+	0    1    1    0
+$EndComp
+Text Label 30750 28300 2    60   ~ 0
+GND
+Wire Wire Line
+	33100 27600 32650 27600
+Wire Wire Line
+	31300 27700 31000 27700
+Wire Wire Line
+	31000 27700 31000 28100
+Wire Wire Line
+	31000 28100 32950 28100
+Wire Wire Line
+	32950 28100 32950 27600
+Connection ~ 32950 27600
+Wire Wire Line
+	33950 27250 33800 27250
+Wire Wire Line
+	33800 27250 33800 27600
+Wire Wire Line
+	33800 27600 33600 27600
+Wire Wire Line
+	32650 27500 33800 27500
+Connection ~ 33800 27500
+Wire Wire Line
+	31300 27800 31200 27800
+Wire Wire Line
+	31200 27800 31200 28300
+Wire Wire Line
+	31200 28300 30750 28300
 Wire Wire Line
-	27900 7800 27800 7800
+	32650 27700 33100 27700
 Wire Wire Line
-	11750 6950 11850 6950
+	33100 27700 33100 28000
 Wire Wire Line
-	11850 7050 11750 7050
+	32650 27800 33050 27800
+Wire Wire Line
+	33050 27800 33050 28100
+Wire Notes Line
+	26950 24950 36150 24950
+Wire Notes Line
+	36150 24950 36150 31150
+Wire Notes Line
+	36150 31150 26950 31150
+Wire Notes Line
+	26950 31150 26950 24950
+Text Notes 29600 25400 0    139  ~ 0
+25Pxx Serial Flash 2
+Text Label 30300 6250 0    60   ~ 0
+V3.3
+Wire Wire Line
+	29900 6100 30150 6100
+Wire Wire Line
+	30150 6100 30150 6250
+Wire Wire Line
+	30150 6250 30300 6250
+Wire Wire Line
+	26300 8100 26050 8100
+Wire Wire Line
+	26050 8200 26300 8200
 $Comp
-L CONN_4X2 P1
-U 1 1 561BD723
-P 27400 7850
-F 0 "P1" H 27400 8100 50  0000 C CNN
-F 1 "CONN_4X2" V 27400 7850 40  0000 C CNN
-F 2 "~" H 27400 7850 60  0000 C CNN
-F 3 "~" H 27400 7850 60  0000 C CNN
-	1    27400 7850
+L CONN_4 P1
+U 1 1 56A36069
+P 26650 8150
+F 0 "P1" V 26600 8150 50  0000 C CNN
+F 1 "FPGA PINS" V 26700 8150 50  0000 C CNN
+F 2 "" H 26650 8150 60  0000 C CNN
+F 3 "" H 26650 8150 60  0000 C CNN
+	1    26650 8150
 	1    0    0    -1
 $EndComp
-Text Label 28000 8000 0    60   ~ 0
-+8Vi
-Text Label 28000 7900 0    60   ~ 0
-GND
-Wire Wire Line
-	28000 7900 27800 7900
 Wire Wire Line
-	27800 8000 28000 8000
+	26300 8000 26050 8000
 $EndSCHEMATC

Commit message: logic-board: S6LX9 R2 first gerbers
Imported from original project folder:
  21-02-2016 2246

14 files changed, 67271 insertions(+), 6747 deletions(-)
Parts:
- removed Jx1, Jx2: USB_2, symbol USB_2
- removed P1: FPGA PINS, symbol CONN_4
- removed P6, P7: CONN_1, symbol CONN_1
- removed R37: 10K, symbol R
- removed R38: 10k, symbol R
- added ???: PIC18F2520-28QFN, ~, symbol PIC18F2520-28QFN
- added P1: FPGA PINS, symbol CONN_5
- added P3: USB_Header, ~, symbol CONN_4X2
- added Q3, Q?: ^^NPN-SOT23, ~, symbol ^^NPN-SOT23
- added R32, R?: 470, symbol R
- added R? (x2): 10k, symbol R
- added SW?: FLASH/RUN, symbol SW_PUSH
Connections:
- net labels added: CH341A_USB_p1, CH341A_USB_p2, CH341A_USB_p3, CH341A_USB_p4, FT232_USB_p1, FT232_USB_p2, FT232_USB_p3, FT232_USB_p4
- net labels removed: FLASH_CS, FLASH_SI
- wire segments 950 -> 982
Other:
- note added: "CH341A / FT232 USB Header"
- note added: "OLD: flash select button RB3"
- moved on the sheet: P5

Commit message: logic-board: MAC10 REV 2.0 - final gerbers, BOM and schematic
Imported from original project folder:
  FPGA_S6LX9_R2

18 files changed, 438793 insertions(+), 30159 deletions(-)
Parts:
- removed P15: DC IN, ~, symbol CONN_2
- removed Q3: ^^NPN-SOT23, ~, symbol ^^NPN-SOT23
- removed R10, R27: 10k, symbol R
- removed R32: 470, symbol R
- removed SW4: FLASH/RUN, symbol SW_PUSH
- removed U3: PIC18F1330, symbol PIC18F1330
- added C23: 0.1 uF, symbol C
- added P10, P11, P12, P6, P7, P9: CONN_1, symbol CONN_1
- added P4: BUTS, ~, symbol CONN_3
- gave numbers to parts that had none: 6
Connections:
- net labels added: FLASHRUNline, PROG_Bline
- wire segments 982 -> 945
Other:
- note added: "EMF Shield"
- note added: "MUST INSTALL R41 to GND (as below) for correct operation"
- note added: "USE 10K RESISTORS for R17 and R13 for correct operation."
- note removed: "OLD: flash select button"
- moved on the sheet: C3, P5, Q3, R10, R27, R32, SW4, U3
